File: Hardware/SparkFun_IoT_Node_LoRaWAN.kicad_sch (KiCad schematic)
At the start: 67 parts, among them J1 USB_C_Receptacle, J2 Conn_01x03, J3 USB_C_Receptacle, J4 SWD, SW1 DPDT_Slide_SMD_7.2x3.5mm, U1 RP2350A, U2 W25Q128JVPIM, U3 APS6404L-3SQR-ZR, U4 XBLR, U5 CH340C, Y1 12MHz

Commit message: Design review updates
Fix typo in USB calculations
Space out buttons in schematic
Add courtyard to flash memory
Reposition measures outside of enclosure outline
Reposition LEd silk outside of light pipe footprint
Other:
- note added: "Differential pair calculation: Conductor Width: 0.2326mm Conductor Spacing 0.127mm Height: 0.2104mm Dielectric Constant: 4.6 Impedance: 89.999 Ohms Computed with Saturn PCB Toolkit"
- note removed: "Differential pair calculation: Conducto Width: 0.2326mm Conductor Spacing 0.127mm Height: 0.2104mm Dielectric Constant: 4.6 Impedance: 89.999 Ohms Computed with Saturn PCB Toolkit"
Changed lines of the file:
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@@
 		)
 	)
-	(text "Differential pair calculation:\nConducto Width: 0.2326mm\nConductor Spacing 0.127mm\nHeight: 0.2104mm\nDielectric Constant: 4.6\nImpedance: 89.999 Ohms\nComputed with Saturn PCB Toolkit"
+	(text "Differential pair calculation:\nConductor Width: 0.2326mm\nConductor Spacing 0.127mm\nHeight: 0.2104mm\nDielectric Constant: 4.6\nImpedance: 89.999 Ohms\nComputed with Saturn PCB Toolkit"
 		(exclude_from_sim no)
 		(at 92.71 35.56 0)
@@
 		)
 	)
-	(text "Differential pair calculation:\nConducto Width: 0.2326mm\nConductor Spacing 0.127mm\nHeight: 0.2104mm\nDielectric Constant: 4.6\nImpedance: 89.999 Ohms\nComputed with Saturn PCB Toolkit"
+	(text "Differential pair calculation:\nConductor Width: 0.2326mm\nConductor Spacing 0.127mm\nHeight: 0.2104mm\nDielectric Constant: 4.6\nImpedance: 89.999 Ohms\nComputed with Saturn PCB Toolkit"
 		(exclude_from_sim no)
 		(at 307.34 35.56 0)
@@
 		(on_board yes)
 		(dnp no)
+		(fields_autoplaced yes)
 		(property "Reference" "JP3"
 			(at 250.19 68.58 0)

Commit message: Design review updates
Move text for D1 and D3 to not overlap wire
Add regulator max output current
Add battery charge current
Add (R) to LoRaWAN silkscreen
Name copper zones
Nudge mesaure text on let side to not overlap lines
Add measures from center to edge of board
Changed lines of the file:
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@@
 		(on_board yes)
 		(dnp no)
-		(fields_autoplaced yes)
 		(property "Reference" "D3"
-			(at 309.88 62.2299 0)
+			(at 313.69 62.23 0)
 			(effects
 				(font
@@
 		)
 		(property "Value" "DT1042-04SO"
-			(at 309.88 64.7699 0)
+			(at 313.69 64.77 0)
 			(effects
 				(font
@@
 		(on_board yes)
 		(dnp no)
-		(fields_autoplaced yes)
 		(property "Reference" "D1"
-			(at 91.44 62.2299 0)
+			(at 95.25 62.23 0)
 			(effects
 				(font
@@
 		)
 		(property "Value" "DT1042-04SO"
-			(at 91.44 64.7699 0)
+			(at 95.25 64.77 0)
 			(effects
 				(font
